File: kimchi_display_lid.sch (KiCad schematic (older format))
At the start: 36 parts, among them J1 DF40HC(3.5)-60DS, J2 DF40HC(3.5)-60DS, J3 H19C-6S-0.5SH, J4 FH19C-40S-0.5SH(10), J5 USB_A, U1 24C32, U2 AP3019AKTR-G1, U3 TXS0108EPW, U4 LSM9DS1

Commit message: Add ESD protection and filtering to USB and DSI
Signed-off-by: Michael Welling <mwelling@ieee.org>
Parts:
- added C10: .1uF, Capacitor_SMD:C_0603_1608Metric, symbol Device:C
- added C9: 100uF, Capacitor_SMD:C_1206_3216Metric, symbol Device:C
- added L2, L3, L4, L5, L6: LCFE121002, kimchi_ulid:LCFE121002, symbol kimchi_ulid:LCFE121002
- added U5: TPD3S014, Package_TO_SOT_SMD:SOT-23-6, symbol Power_Protection:TPD3S014
Connections:
- net labels added: DISP1_CK_N, DISP1_CK_P, DISP1_D0_N, DISP1_D0_P, DISP1_D1_N, DISP1_D1_P, DISP1_D2_N, DISP1_D2_P, DISP1_D3_N, DISP1_D3_P, VBUS
- net labels removed: USB2_ID, USB2_VBUS
- wire segments 214 -> 250

Commit message: Whooops PWM is on GPIO1_13
Signed-off-by: Michael Welling <mwelling@ieee.org>
Changed lines of the file:
@@
 Text Notes 10800 9000 0    50   ~ 0
 NOTE: CONNECTORS INTENTIONALLY MIRRORED TO COMPENSATE\nFOR DIFFERENT PIN 1 CONVENTIONS ON THE CONNECTOR\nVERSUS THE FPC ON THE DISPLAY
-Text Label 4000 5900 0    50   ~ 0
+Text Label 4000 5800 0    50   ~ 0
 BL_PWM
 Text Label 4000 5300 0    50   ~ 0
@@
 Text Notes 2700 4200 0    100  ~ 0
 LEVEL TRANSLATOR
-Text Notes 2000 5950 0    40   ~ 0
+Text Notes 2000 5850 0    40   ~ 0
 PWM2_OUT =>
 $Comp
@@
 Text Label 4000 5700 0    50   ~ 0
 INT_M
-Text Label 4000 5800 0    50   ~ 0
+Text Label 4000 5900 0    50   ~ 0
 INT1A_G
 Text Label 4000 5200 0    50   ~ 0

Commit message: Move the mounting holes to avoid blocking LCD FPC
Also removes a bit length on the board to compensate for
the cable wrapping around the PCB.

May have to move the touchsreen connector and use an adapter
to add length.

Signed-off-by: Michael Welling <mwelling@ieee.org>
Parts:
- J5: symbol Connector:USB_A -> kimchi_display_lid-rescue:USB_A-Connector
Changed lines of the file:
@@
 PWM2_OUT =>
 $Comp
-L Connector:USB_A J5
+L kimchi_display_lid-rescue:USB_A-Connector J5
 U 1 1 6009A0A2
 P 14550 6700

Commit message: Add part numbers to the schematic for BOM export
Signed-off-by: Michael Welling <mwelling@ieee.org>
Parts:
- C1: Part (none) -> C0603C105K4PAC7411
- C10, C3, C4, C6, C7: Part (none) -> C0603C104M5RACAUTO
- C2: Part (none) -> CGA3E3X7R1H224K080AB
- C5, C8: Part (none) -> CL10A106MP8NNNC
- C9: Part (none) -> CC1206MKX5R5BB107
- J3: Part (none) -> H19C-6S-0.5SH
- J4: Part (none) -> FH19C-40S-0.5SH(10)
- J5: Part (none) -> 1-292303-6
- L2, L3, L4, L5, L6: Part (none) -> LCFE121002
- R1: Part (none) -> RE0603FRE0710RL
- R2, R3, R4, R5, R6, R7, R8: Part (none) -> RC0603JR-074K7L
- U3: Part (none) -> TXS0108EPW
- U4: Part (none) -> LSM9DS1
- U5: Part (none) -> TPD3S014
Changed lines of the file:
@@
 F 2 "Resistor_SMD:R_0603_1608Metric" V 8480 9700 50  0001 C CNN
 F 3 "~" H 8550 9700 50  0001 C CNN
+F 4 "RE0603FRE0710RL" H 8550 9700 50  0001 C CNN "Part"
 	1    8550 9700
 	1    0    0    -1
@@
 F 2 "Capacitor_SMD:C_0603_1608Metric" H 6938 9400 50  0001 C CNN
 F 3 "~" H 6900 9550 50  0001 C CNN
+F 4 "C0603C105K4PAC7411" H 6900 9550 50  0001 C CNN "Part"
 	1    6900 9550
 	1    0    0    -1
@@
 F 2 "Capacitor_SMD:C_0603_1608Metric" H 9288 9500 50  0001 C CNN
 F 3 "~" H 9250 9650 50  0001 C CNN
+F 4 "CGA3E3X7R1H224K080AB" H 9250 9650 50  0001 C CNN "Part"
 	1    9250 9650
 	1    0    0    -1
@@
 F 2 "kimchi_ulid:HRS_FH19C-40S-0.5SH_1x40-1MP_P0.50mm" H 10500 7650 50  0001 C CNN
 F 3 "~" H 10500 7650 50  0001 C CNN
+F 4 "FH19C-40S-0.5SH(10)" H 10500 7650 50  0001 C CNN "Part"
 	1    10500 7650
 	1    0    0    1
@@
 F 2 "kimchi_ulid:HRS_FH19C-6S-0.5SH_1x06-1MP_P0.50mm" H 8150 6550 50  0001 C CNN
 F 3 "~" H 8150 6550 50  0001 C CNN
+F 4 "H19C-6S-0.5SH" H 8150 6550 50  0001 C CNN "Part"
 	1    8150 6550
 	1    0    0    1
@@
 F 2 "Resistor_SMD:R_0603_1608Metric" V 7280 5950 50  0001 C CNN
 F 3 "~" H 7350 5950 50  0001 C CNN
+F 4 "RC0603JR-074K7L" H 7350 5950 50  0001 C CNN "Part"
 	1    7350 5950
 	1    0    0    -1
@@
 F 2 "Resistor_SMD:R_0603_1608Metric" V 7580 5950 50  0001 C CNN
 F 3 "~" H 7650 5950 50  0001 C CNN
+F 4 "RC0603JR-074K7L" H 7650 5950 50  0001 C CNN "Part"
 	1    7650 5950
 	1    0    0    -1
@@
 F 2 "Package_SO:TSSOP-20_4.4x6.5mm_P0.65mm" H 3450 4750 50  0001 C CNN
 F 3 "www.ti.com/lit/ds/symlink/txs0108e.pdf" H 3450 5400 50  0001 C CNN
+F 4 "TXS0108EPW" H 3450 5500 50  0001 C CNN "Part"
 	1    3450 5500
 	1    0    0    -1
@@
 F 2 "Capacitor_SMD:C_0603_1608Metric" H 4188 4450 50  0001 C CNN
 F 3 "~" H 4150 4600 50  0001 C CNN
+F 4 "C0603C104M5RACAUTO" H 4150 4600 50  0001 C CNN "Part"
 	1    4150 4600
 	-1   0    0    1
@@
 F 2 "Capacitor_SMD:C_0603_1608Metric" H 2338 4450 50  0001 C CNN
 F 3 "~" H 2300 4600 50  0001 C CNN
+F 4 "C0603C104M5RACAUTO" H 2300 4600 50  0001 C CNN "Part"
 	1    2300 4600
 	1    0    0    -1
@@
 F 2 "Resistor_SMD:R_0603_1608Metric" V 2680 4700 50  0001 C CNN
 F 3 "~" H 2750 4700 50  0001 C CNN
+F 4 "RC0603JR-074K7L" H 2750 4700 50  0001 C CNN "Part"
 	1    2750 4700
 	1    0    0    -1
@@
 F 2 "kimchi_ulid:TE_1-292303-6" H 14700 6650 50  0001 C CNN
 F 3 " ~" H 14700 6650 50  0001 C CNN
+F 4 "1-292303-6" H 14550 6700 50  0001 C CNN "Part"
 	1    14550 6700
 	-1   0    0    -1
@@
 F 7 "LSM9DS1" H 3450 8450 50  0001 L BNN "Field7"
 F 8 "Unavailable" H 3450 8450 50  0001 L BNN "Field8"
+F 9 "LSM9DS1" H 3450 8450 50  0001 C CNN "Part"
 	1    3450 8450
 	1    0    0    -1
@@
 F 2 "Resistor_SMD:R_0603_1608Metric" V 2080 7350 50  0001 C CNN
 F 3 "~" H 2150 7350 50  0001 C CNN
+F 4 "RC0603JR-074K7L" H 2150 7350 50  0001 C CNN "Part"
 	1    2150 7350
 	-1   0    0    1
@@
 F 2 "Resistor_SMD:R_0603_1608Metric" V 2280 7350 50  0001 C CNN
 F 3 "~" H 2350 7350 50  0001 C CNN
+F 4 "RC0603JR-074K7L" H 2350 7350 50  0001 C CNN "Part"
 	1    2350 7350
 	-1   0    0    1
@@
 F 2 "Resistor_SMD:R_0603_1608Metric" V 1680 7350 50  0001 C CNN
 F 3 "~" H 1750 7350 50  0001 C CNN
+F 4 "RC0603JR-074K7L" H 1750 7350 50  0001 C CNN "Part"
 	1    1750 7350
 	1    0    0    -1
@@
 F 2 "Resistor_SMD:R_0603_1608Metric" V 1880 7350 50  0001 C CNN
 F 3 "~" H 1950 7350 50  0001 C CNN
+F 4 "RC0603JR-074K7L" H 1950 7350 50  0001 C CNN "Part"
 	1    1950 7350
 	1    0    0    -1
@@
 F 2 "Capacitor_SMD:C_0603_1608Metric" H 1938 9250 50  0001 C CNN
 F 3 "~" H 1900 9400 50  0001 C CNN
+F 4 "CL10A106MP8NNNC" H 1900 9400 50  0001 C CNN "Part"
 	1    1900 9400
 	1    0    0    -1
@@
 F 2 "Capacitor_SMD:C_0603_1608Metric" H 2338 9250 50  0001 C CNN
 F 3 "~" H 2300 9400 50  0001 C CNN
+F 4 "C0603C104M5RACAUTO" H 2300 9400 50  0001 C CNN "Part"
 	1    2300 9400
 	1    0    0    -1
@@
 F 2 "Capacitor_SMD:C_0603_1608Metric" H 5288 7850 50  0001 C CNN
 F 3 "~" H 5250 8000 50  0001 C CNN
+F 4 "CL10A106MP8NNNC" H 5250 8000 50  0001 C CNN "Part"
 	1    5250 8000
 	1    0    0    -1
@@
 F 2 "Capacitor_SMD:C_0603_1608Metric" H 4888 7850 50  0001 C CNN
 F 3 "~" H 4850 8000 50  0001 C CNN
+F 4 "C0603C104M5RACAUTO" H 4850 8000 50  0001 C CNN "Part"
 	1    4850 8000
 	1    0    0    -1
@@
 F 2 "Package_TO_SOT_SMD:SOT-23-6" H 13100 6350 50  0001 C CNN
 F 3 "http://www.ti.com/lit/ds/symlink/tpd3s014.pdf" H 12900 6250 50  0001 C CNN
+F 4 "TPD3S014" H 13100 6000 50  0001 C CNN "Part"
 	1    13100 6000
 	1    0    0    -1
@@
 F 2 "Capacitor_SMD:C_1206_3216Metric" H 13838 6900 50  0001 C CNN
 F 3 "~" H 13800 7050 50  0001 C CNN
+F 4 "CC1206MKX5R5BB107" H 13800 7050 50  0001 C CNN "Part"
 	1    13800 7050
 	1    0    0    -1
@@
 F 2 "Capacitor_SMD:C_0603_1608Metric" H 12288 5950 50  0001 C CNN
 F 3 "~" H 12250 6100 50  0001 C CNN
+F 4 "C0603C104M5RACAUTO" H 12250 6100 50  0001 C CNN "Part"
 	1    12250 6100
 	-1   0    0    1
@@
 F 2 "kimchi_ulid:LCFE121002" H 8700 8100 50  0001 C CNN
 F 3 "~" H 8700 8100 50  0001 C CNN
+F 4 "LCFE121002" H 8700 8100 50  0001 C CNN "Part"
 	1    8700 8100
 	-1   0    0    -1
@@
 F 2 "kimchi_ulid:LCFE121002" H 8700 8400 50  0001 C CNN
 F 3 "~" H 8700 8400 50  0001 C CNN
+F 4 "LCFE121002" H 8700 8400 50  0001 C CNN "Part"
 	1    8700 8400
 	-1   0    0    -1
@@
 F 2 "kimchi_ulid:LCFE121002" H 8700 8700 50  0001 C CNN
 F 3 "~" H 8700 8700 50  0001 C CNN
+F 4 "LCFE121002" H 8700 8700 50  0001 C CNN "Part"
 	1    8700 8700
 	-1   0    0    -1
@@
 F 2 "kimchi_ulid:LCFE121002" H 8700 9000 50  0001 C CNN
 F 3 "~" H 8700 9000 50  0001 C CNN
+F 4 "LCFE121002" H 8700 9000 50  0001 C CNN "Part"
 	1    8700 9000
 	-1   0    0    -1
@@
 F 2 "kimchi_ulid:LCFE121002" H 8700 7800 50  0001 C CNN
 F 3 "~" H 8700 7800 50  0001 C CNN
+F 4 "LCFE121002" H 8700 7800 50  0001 C CNN "Part"
 	1    8700 7800
 	-1   0    0    -1

Commit message: IMU Changed
9DOF IMU is out of stock, added new IMU that is 6DOF adjusted PCB design to include new IMU.
Parts:
- removed C5: 10uF, Capacitor_SMD:C_0603_1608Metric, symbol Device:C
- removed C6: .1uF, Capacitor_SMD:C_0603_1608Metric, symbol Device:C
- removed U4: LSM9DS1, PQFN24P43_350X300X102L35X23N, symbol kimchi_ulid:LSM9DS1_LSM9DS1
- added U4: LSM6DSRTR, kimchi_ulid:LSM6DSRTR, symbol kimchi_ulid:LSM6DSRTR
- C1, C10, C2, C3, C4, C7, C8, C9: symbol Device:C -> kimchi_display_lid-rescue:C-Device
- H1, H2, H3, H4, H5, H6, H7, H8: symbol Mechanical:MountingHole_Pad -> kimchi_display_lid-rescue:MountingHole_Pad-Mechanical
- L1: symbol Device:L_Small -> kimchi_display_lid-rescue:L_Small-Device
- LOGO1, LOGO2: symbol Graphic:Logo_Open_Hardware_Small -> kimchi_display_lid-rescue:Logo_Open_Hardware_Small-Graphic
- R1, R2, R3, R4, R5, R6, R7, R8: symbol Device:R -> kimchi_display_lid-rescue:R-Device
Connections:
- wire segments 250 -> 243
Other:
- note added: "6DOF IMU"
- note removed: "9DOF IMU"

Commit message: Logos
added logots
Parts:
- added L?: GG_LOGO, kimchi_ulid:groupgets_logo, symbol kimchi_ulid:GG_LOGO
- added L?: OSHPARK_LOGO, kimchi_ulid:oshpark_logo, symbol kimchi_ulid:OSHPARK_LOGO
Changed lines of the file:
@@
 Wire Wire Line
 	2350 8850 2350 7400
+$Comp
+L kimchi_ulid:GG_LOGO L?
+U 1 1 601047E2
+P 13350 3700
+F 0 "L?" H 13400 3745 50  0000 L CNN
+F 1 "GG_LOGO" H 13400 3654 50  0000 L CNN
+F 2 "kimchi_ulid:groupgets_logo" H 13350 3700 50  0001 C CNN
+F 3 "" H 13350 3700 50  0001 C CNN
+	1    13350 3700
+	1    0    0    -1
+$EndComp
+$Comp
+L kimchi_ulid:OSHPARK_LOGO L?
+U 1 1 60105FC2
+P 13400 3900
+F 0 "L?" H 13450 3945 50  0000 L CNN
+F 1 "OSHPARK_LOGO" H 13450 3854 50  0000 L CNN
+F 2 "kimchi_ulid:oshpark_logo" H 13400 3900 50  0001 C CNN
+F 3 "" H 13400 3900 50  0001 C CNN
+	1    13400 3900
+	1    0    0    -1
+$EndComp
 $EndSCHEMATC
